File: PCB Files/kiCad/Step_Direction_Board.kicad_pcb (KiCad board)
At the start: 2 copper layers, 65 x 19.5 mm, 15 parts, among them J0 Conn_01x02, U0 SN75451BDR, U1 SN75451BDR, U2 SN75451BDR, U3 SN75451BDR

Commit message: let's try this again
Parts:
- removed J0, SDI0, SDI1, SDI2, SDI3: Conn_01x02, Connector_PinHeader_2.54mm:PinHeader_1x02_P2.54mm_Horizontal
- added C0: 0.1uF, Capacitor_SMD:C_0805_2012Metric_Pad1.15x1.40mm_HandSolder, B.Cu at (127.8, 113.1)
- added C1: 0.1uF, Capacitor_SMD:C_0805_2012Metric_Pad1.15x1.40mm_HandSolder, B.Cu at (140.0, 114.1)
- added C2: 0.1uF, Capacitor_SMD:C_0805_2012Metric_Pad1.15x1.40mm_HandSolder, B.Cu at (153.0, 114.1)
- added C3: 0.1uF, Capacitor_SMD:C_0805_2012Metric_Pad1.15x1.40mm_HandSolder, B.Cu at (166.1, 114.1)
- added J1: Conn_01x06, Connector_PinHeader_2.54mm:PinHeader_1x06_P2.54mm_Horizontal, F.Cu at (132.5, 109.2)
- added J2: Conn_01x06, Connector_PinHeader_2.54mm:PinHeader_1x06_P2.54mm_Horizontal, F.Cu at (160.8, 109.2)
Connections:
- net Net-(SDI0-Pad1) renamed /LS0/in1
- net Net-(SDI0-Pad2) renamed /LS0/in2
- net Net-(SDI1-Pad1) renamed /LS1/in1
- net Net-(SDI1-Pad2) renamed /LS1/in2
- net Net-(SDI2-Pad1) renamed /LS2/in1
- net Net-(SDI2-Pad2) renamed /LS2/in2
- net Net-(SDI3-Pad1) renamed /LS3/in1
- net Net-(SDI3-Pad2) renamed /LS3/in2
Routing:
- net GND: track 0.00 -> 14.0 mm
- net 5v: track 112.6 -> 117.6 mm
- net /LS1/in2: track 4.76 -> 8.31 mm
- net /LS2/in2: track 4.76 -> 6.84 mm
- net /LS3/in2: track 4.76 -> 6.58 mm
- net /LS1/in1: track 9.02 -> 10.6 mm
- net /LS0/in2: track 4.76 -> 6.29 mm
- net /LS2/in1: track 9.02 -> 10.1 mm
Other:
- board size 65 x 19.5 mm -> 66 x 21.5 mm
- net class Default: trace_width 0.5 -> 0.7
- board text added: "D"
- board text added: "D0"
- board text added: "D1"
- board text added: "D2"
- board text added: "D3"
- board text added: "NC"
- board text added: "S"
- board text added: "S0"
- board text added: "S1"
- board text added: "S2"
- board text added: "S3"
- board text removed: "Dir"
- board text removed: "Step"
